File: Hardware/PCB/ao_dc_mixer/ao_dc_mixer.kicad_pcb (KiCad board)
At the start: 2 copper layers, 0 parts

Commit message: PCB and panel design
Parts:
- added C1: 100 pF, ao_tht:C_Disc_D3.0mm_W1.6mm_P2.50mm, F.Cu at (132.9, 91.0)
- added C2: 10uF, ao_tht:CP_Radial_D5.0mm_P2.00mm, F.Cu at (117.6, 83.3)
- added C3: 10uF, ao_tht:CP_Radial_D5.0mm_P2.00mm, F.Cu at (119.6, 108.7)
- added C4: 330 pF, ao_tht:C_Disc_D3.0mm_W1.6mm_P2.50mm, F.Cu at (153.2, 108.7)
- added C5: 0.1uF, ao_tht:C_Disc_D3.0mm_W1.6mm_P2.50mm, F.Cu at (132.9, 96.0)
- added C6: 0.1uF, ao_tht:C_Disc_D3.0mm_W1.6mm_P2.50mm, F.Cu at (153.2, 96.0)
- added C7: 330 pF, ao_tht:C_Disc_D3.0mm_W1.6mm_P2.50mm, F.Cu at (153.2, 83.3)
- added D1: 2N5817, ao_tht:D_DO-41_SOD81_P7.62mm_Horizontal, F.Cu at (112.5, 83.3)
- added D2: 2N5817, ao_tht:D_DO-41_SOD81_P7.62mm_Horizontal, F.Cu at (112.5, 101.1)
- added D3: 1N4148, ao_tht:D_DO-35_SOD27_P7.62mm_Horizontal, F.Cu at (106.2, 118.9)
- added D4: 1N4148, ao_tht:D_DO-35_SOD27_P7.62mm_Horizontal, F.Cu at (110.0, 126.5)
- added G***: LOGO, ao_dc_mixer:ao_dc_mixer_slide_holes, B.Cu at (130.0, 130.0)
- added H1: MountingHole, ao_tht:MountingHole_3.2mm_M3, F.Cu at (100.0, 155.0)
- added H2: MountingHole, ao_tht:MountingHole_3.2mm_M3, F.Cu at (160.0, 155.0)
- added J1: Conn_01x02, ao_tht:Molex_KK-254_AE-6410-02A_1x02_P2.54mm_Vertical, F.Cu at (157.0, 59.9)
- added J2: Conn_01x02, ao_tht:Molex_KK-254_AE-6410-02A_1x02_P2.54mm_Vertical, F.Cu at (141.5, 59.9)
- added J3: Conn_01x02, ao_tht:Molex_KK-254_AE-6410-02A_1x02_P2.54mm_Vertical, F.Cu at (126.5, 59.9)
- added J4: Synth_power_2x5, ao_tht:Power_Header, F.Cu at (104.9, 101.1)
- added J5: Conn_01x02, ao_tht:Molex_KK-254_AE-6410-02A_1x02_P2.54mm_Vertical, F.Cu at (109.2, 153.4)
- added J6: Conn_01x02, ao_tht:Molex_KK-254_AE-6410-02A_1x02_P2.54mm_Vertical, F.Cu at (124.1, 153.4)
- added N1: AO logo, ao_tht:analogoutput, F.Cu at (139.2, 75.7)
- added N2: OSHW logo, Symbol:OSHW-Logo2_7.3x6mm_SilkScreen, F.Cu at (106.5, 75.5)
- added R1: 120k, ao_tht:R_Axial_DIN0207_L6.3mm_D2.5mm_P7.62mm_Horizontal, F.Cu at (157.0, 118.9)
- added R10: 10k, ao_tht:R_Axial_DIN0207_L6.3mm_D2.5mm_P7.62mm_Horizontal, F.Cu at (150.7, 101.1)
- added R11: 10k, ao_tht:R_Axial_DIN0207_L6.3mm_D2.5mm_P7.62mm_Horizontal, F.Cu at (132.9, 101.1)
- added R12: 10k, ao_tht:R_Axial_DIN0207_L6.3mm_D2.5mm_P7.62mm_Horizontal, F.Cu at (125.2, 104.9)
- added R13: 10k, ao_tht:R_Axial_DIN0207_L6.3mm_D2.5mm_P7.62mm_Horizontal, F.Cu at (158.3, 104.9)
- added R14: 1k, ao_tht:R_Axial_DIN0207_L6.3mm_D2.5mm_P7.62mm_Horizontal, F.Cu at (158.3, 112.5)
- added R15: 10k, ao_tht:R_Axial_DIN0207_L6.3mm_D2.5mm_P7.62mm_Horizontal, F.Cu at (150.7, 91.0)
- added R16: 10k, ao_tht:R_Axial_DIN0207_L6.3mm_D2.5mm_P7.62mm_Horizontal, F.Cu at (158.3, 87.2)
- added R17: 1k, ao_tht:R_Axial_DIN0207_L6.3mm_D2.5mm_P7.62mm_Horizontal, F.Cu at (158.3, 79.5)
- added R2: 120k, ao_tht:R_Axial_DIN0207_L6.3mm_D2.5mm_P7.62mm_Horizontal, F.Cu at (141.8, 118.9)
- added R3: 120k, ao_tht:R_Axial_DIN0207_L6.3mm_D2.5mm_P7.62mm_Horizontal, F.Cu at (127.8, 118.9)
- added R6: 15k, ao_tht:R_Axial_DIN0207_L6.3mm_D2.5mm_P7.62mm_Horizontal, F.Cu at (125.2, 87.2)
- added R7: 15k, ao_tht:R_Axial_DIN0207_L6.3mm_D2.5mm_P7.62mm_Horizontal, F.Cu at (98.6, 126.5)
- added R8: 68k, ao_tht:R_Axial_DIN0207_L6.3mm_D2.5mm_P7.62mm_Horizontal, F.Cu at (102.4, 118.9)
- added R9: 15k, ao_tht:R_Axial_DIN0207_L6.3mm_D2.5mm_P7.62mm_Horizontal, F.Cu at (113.8, 126.5)
- added RV1: B100k, ao_tht:Potentiometer_Alpha_RA6020F_Single_Slide, B.Cu at (162.0, 135.0)
- added RV2: B100k, ao_tht:Potentiometer_Alpha_RA6020F_Single_Slide, B.Cu at (147.0, 135.0)
- added RV3: B100k, ao_tht:Potentiometer_Alpha_RA6020F_Single_Slide, B.Cu at (132.0, 135.0)
- added RV4: B100k, ao_tht:Potentiometer_Alpha_RA6020F_Single_Slide, B.Cu at (102.0, 135.0)
- added RV5: 10k, ao_tht:Potentiometer_Bourns_3296W_Vertical, F.Cu at (125.2, 75.7)
- added RV6: B100k, ao_tht:Potentiometer_Alpha_RA6020F_Single_Slide, B.Cu at (117.0, 135.0)
- added U3: TL074, ao_tht:DIP-14_W7.62mm_Socket_LongPads, F.Cu at (137.9, 88.4)
Routing:
- net /~OUT: track 0.00 -> 118.7 mm
- net Net-(C1-Pad2): track 0.00 -> 84.3 mm
- net Net-(RV5-Pad1): track 0.00 -> 83.9 mm
- net /OUT: track 0.00 -> 83.5 mm
- net -12V: track 0.00 -> 78.4 mm
- net Net-(C1-Pad1): track 0.00 -> 68.1 mm
- net /V_BIAS: track 0.00 -> 63.4 mm
- net +12V: track 0.00 -> 53.4 mm
- net Net-(R12-Pad1): track 0.00 -> 28.6 mm
- net Net-(R1-Pad2): track 0.00 -> 14.6 mm
- net Net-(R7-Pad1): track 0.00 -> 14.1 mm
- net Net-(R3-Pad2): track 0.00 -> 13.8 mm
- net Net-(C7-Pad1): track 0.00 -> 13.8 mm
- net Net-(C4-Pad1): track 0.00 -> 13.8 mm
- net Net-(R2-Pad2): track 0.00 -> 13.6 mm
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- added copper zone on B.Cu, net GND
- added copper zone on F.Cu, net GND
Other:
- board outline added: 74 x 103 mm
- net class Power added: clearance 0.2, trace_width 0.75, via_dia 0.8, via_drill 0.4
- board text added: "DC Mixer"
- board text added: "Rich Holmes Mar 2021 CC0 1.0 Universal"

Commit message: Various revisions, new DNF symbols
Parts:
- removed C1: 100 pF, ao_tht:C_Disc_D3.0mm_W1.6mm_P2.50mm
Routing:
- net Net-(R1-Pad1): track 68.1 -> 71.0 mm

Commit message: Gerbers, BOM, final version before fabrication
Parts:
- removed G***: LOGO, ao_dc_mixer:ao_dc_mixer_slide_holes
- removed N1: AO logo, ao_tht:analogoutput
- removed N2: OSHW logo, Symbol:OSHW-Logo2_7.3x6mm_SilkScreen
- added GRAF1: AO Logo, ao_tht:analogoutput, F.Cu at (142.0, 74.0)
- added GRAF2: OSHW Logo, ao_tht:OSHW-Logo2_7.3x6mm_SilkScreen, F.Cu at (107.0, 79.8)
- added GRAF3: Panel holes, ao_dc_mixer:ao_dc_mixer_slide_holes, F.Cu at (130.0, 130.0)
- J1, J2, J3, J5, J6: value Conn_01x02 -> 2 Pin Molex Header
- moved J1 5.08 mm to (157.0, 65.0)
- moved J2 5.08 mm to (141.5, 65.0)
- moved J3 5.08 mm to (126.5, 65.0)
Routing:
- net /IN1: track 7.13 -> 5.01 mm
- net /IN3: track 7.58 -> 5.49 mm
- net /IN2: track 7.59 -> 5.50 mm
Other:
- board size 74 x 103 mm -> 74 x 97.9 mm
- board text added: "IN1"
- board text added: "IN2"
- board text added: "IN3"
- board text added: "OUT"
- board text added: "~OUT"
